File: Arret_urgence.kicad_pcb (KiCad board)
At the start: 2 copper layers, 30 x 22 mm, 7 parts, among them J1 Conn_01x02, J2 USB_C_Receptacle_USB2.0, J3 USB_C_Receptacle_USB2.0

Commit message: modif schematic
Parts:
- J3: moved to F.Cu
- turned J3 to 180 degrees
Connections:
- J3 pad A5: Net-(J2-PadA5) -> Net-(J2-PadB5)
- J3 pad A6: Net-(J2-PadA6) -> Net-(J2-PadB6)
- J3 pad A7: Net-(J2-PadA7) -> Net-(J2-PadB7)
- J3 pad A8: Net-(J2-PadA8) -> Net-(J2-PadB8)
- J3 pad B5: Net-(J2-PadB5) -> Net-(J2-PadA5)
- J3 pad B6: Net-(J2-PadB6) -> Net-(J2-PadA6)
- J3 pad B7: Net-(J2-PadB7) -> Net-(J2-PadA7)
- J3 pad B8: Net-(J2-PadB8) -> Net-(J2-PadA8)
Routing:
- net +5V: track 36.0 -> 17.9 mm
- net GND: track 77.8 -> 63.6 mm, vias 1 -> 0
- net Net-(J2-PadB8): track 8.03 -> 0.00 mm, vias 1 -> 0
- net Net-(J2-PadA5): track 7.48 -> 0.00 mm, vias 1 -> 0
- net Net-(J2-PadB5): track 7.47 -> 0.00 mm, vias 1 -> 0
- net Net-(J2-PadA8): track 7.28 -> 0.00 mm, vias 1 -> 0
- net Net-(J2-PadB7): track 7.24 -> 0.00 mm, vias 1 -> 0
- net Net-(J2-PadB6): track 6.97 -> 0.00 mm, vias 1 -> 0
- net Net-(J2-PadA6): track 6.80 -> 0.00 mm, vias 1 -> 0
- net Net-(J2-PadA7): track 6.56 -> 0.00 mm, vias 1 -> 0

Commit message: modif
Connections:
- J1 pad 1: +5V -> Net-(J2-PadA4)
- J1 pad 2: +5V -> Net-(J1-Pad2)
- J2 pad A4: +5V -> Net-(J2-PadA4)
- J2 pad A9: +5V -> Net-(J2-PadA4)
- J2 pad B4: +5V -> Net-(J2-PadA4)
- J2 pad B9: +5V -> Net-(J2-PadA4)
- J3 pad A4: +5V -> Net-(J1-Pad2)
- J3 pad A9: +5V -> Net-(J1-Pad2)
- J3 pad B4: +5V -> Net-(J1-Pad2)
- J3 pad B9: +5V -> Net-(J1-Pad2)
Routing:
- net +5V: track 17.9 -> 0.00 mm
- net Net-(J1-Pad2): track 0.00 -> 17.4 mm
- net Net-(J2-PadA4): track 0.00 -> 17.3 mm
- net Net-(J2-PadB5): track 0.00 -> 7.27 mm
- net Net-(J2-PadA7): track 0.00 -> 6.99 mm
- net Net-(J2-PadA8): track 0.00 -> 6.95 mm, vias 0 -> 2
- net Net-(J2-PadB6): track 0.00 -> 6.88 mm, vias 0 -> 2
- net Net-(J2-PadA6): track 0.00 -> 6.79 mm, vias 0 -> 2
- net Net-(J2-PadB8): track 0.00 -> 6.77 mm
- net Net-(J2-PadB7): track 0.00 -> 6.63 mm
- net Net-(J2-PadA5): track 0.00 -> 6.60 mm, vias 0 -> 2
- net GND: track 63.6 -> 68.4 mm
- added copper zone on F.Cu, net GND
