File: Arret_urgence.kicad_sch (KiCad schematic)
At the start: 7 parts, among them J1 Conn_01x02, J2 USB_C_Receptacle_USB2.0, J3 USB_C_Receptacle_USB2.0

Commit message: modif schematic
Connections:
- net at J3.A5 (CC1): now also J2.B5 (CC2); no longer J2.A5 (CC1)
- net at J3.A6 (D+): now also J2.B6 (D+); no longer J2.A6 (D+)
- net at J3.A7 (D-): now also J2.B7 (D-); no longer J2.A7 (D-)
- net at J3.A8 (SBU1): now also J2.B8 (SBU2); no longer J2.A8 (SBU1)
- net at J3.B5 (CC2): now also J2.A5 (CC1); no longer J2.B5 (CC2)
- net at J3.B6 (D+): now also J2.A6 (D+); no longer J2.B6 (D+)
- net at J3.B7 (D-): now also J2.A7 (D-); no longer J2.B7 (D-)
- net at J3.B8 (SBU2): now also J2.A8 (SBU1); no longer J2.B8 (SBU2)
Changed lines of the file:
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@@
+    (stroke (width 0) (type default) (color 0 0 0 0))
+  )
+  (wire (pts (xy 106.68 93.98) (xy 109.22 93.98))
+    (stroke (width 0) (type default) (color 0 0 0 0))
+  )
+  (wire (pts (xy 106.68 90.17) (xy 106.68 88.9))
+    (stroke (width 0) (type default) (color 0 0 0 0))
+  )
+  (wire (pts (xy 106.68 81.28) (xy 109.22 81.28))
     (stroke (width 0) (type default) (color 0 0 0 0))
   )
@@
     (stroke (width 0) (type default) (color 0 0 0 0))
   )
+  (wire (pts (xy 100.33 90.17) (xy 106.68 90.17))
+    (stroke (width 0) (type default) (color 0 0 0 0))
+  )
+  (wire (pts (xy 109.22 87.63) (xy 115.57 87.63))
+    (stroke (width 0) (type default) (color 0 0 0 0))
+  )
+  (wire (pts (xy 107.95 82.55) (xy 115.57 82.55))
+    (stroke (width 0) (type default) (color 0 0 0 0))
+  )
+  (wire (pts (xy 107.95 80.01) (xy 107.95 82.55))
+    (stroke (width 0) (type default) (color 0 0 0 0))
+  )
+  (wire (pts (xy 107.95 87.63) (xy 107.95 90.17))
+    (stroke (width 0) (type default) (color 0 0 0 0))
+  )
+  (wire (pts (xy 100.33 102.87) (xy 107.95 102.87))
+    (stroke (width 0) (type default) (color 0 0 0 0))
+  )
   (wire (pts (xy 138.43 118.11) (xy 134.62 118.11))
     (stroke (width 0) (type default) (color 0 0 0 0))
   )
-  (wire (pts (xy 100.33 92.71) (xy 115.57 92.71))
+  (wire (pts (xy 109.22 80.01) (xy 115.57 80.01))
+    (stroke (width 0) (type default) (color 0 0 0 0))
+  )
+  (wire (pts (xy 109.22 81.28) (xy 109.22 80.01))
+    (stroke (width 0) (type default) (color 0 0 0 0))
+  )
+  (wire (pts (xy 100.33 87.63) (xy 107.95 87.63))
     (stroke (width 0) (type default) (color 0 0 0 0))
   )
@@
     (stroke (width 0) (type default) (color 0 0 0 0))
   )
-  (wire (pts (xy 100.33 102.87) (xy 115.57 102.87))
-    (stroke (width 0) (type default) (color 0 0 0 0))
-  )
-  (wire (pts (xy 100.33 95.25) (xy 115.57 95.25))
+  (wire (pts (xy 107.95 90.17) (xy 115.57 90.17))
+    (stroke (width 0) (type default) (color 0 0 0 0))
+  )
+  (wire (pts (xy 109.22 93.98) (xy 109.22 92.71))
+    (stroke (width 0) (type default) (color 0 0 0 0))
+  )
+  (wire (pts (xy 109.22 104.14) (xy 109.22 102.87))
     (stroke (width 0) (type default) (color 0 0 0 0))
   )
@@
     (stroke (width 0) (type default) (color 0 0 0 0))
   )
+  (wire (pts (xy 100.33 105.41) (xy 106.68 105.41))
+    (stroke (width 0) (type default) (color 0 0 0 0))
+  )
   (wire (pts (xy 81.28 116.84) (xy 85.09 116.84))
     (stroke (width 0) (type default) (color 0 0 0 0))
   )
-  (wire (pts (xy 100.33 80.01) (xy 115.57 80.01))
-    (stroke (width 0) (type default) (color 0 0 0 0))
-  )
-  (wire (pts (xy 100.33 82.55) (xy 115.57 82.55))
-    (stroke (width 0) (type default) (color 0 0 0 0))
-  )
   (wire (pts (xy 113.03 72.39) (xy 113.03 74.93))
     (stroke (width 0) (type default) (color 0 0 0 0))
   )
-  (wire (pts (xy 100.33 90.17) (xy 115.57 90.17))
+  (wire (pts (xy 109.22 92.71) (xy 115.57 92.71))
+    (stroke (width 0) (type default) (color 0 0 0 0))
+  )
+  (wire (pts (xy 100.33 95.25) (xy 106.68 95.25))
     (stroke (width 0) (type default) (color 0 0 0 0))
   )
@@
     (stroke (width 0) (type default) (color 0 0 0 0))
   )
+  (wire (pts (xy 107.95 95.25) (xy 115.57 95.25))
+    (stroke (width 0) (type default) (color 0 0 0 0))
+  )
+  (wire (pts (xy 109.22 88.9) (xy 109.22 87.63))
+    (stroke (width 0) (type default) (color 0 0 0 0))
+  )
+  (wire (pts (xy 106.68 95.25) (xy 106.68 93.98))
+    (stroke (width 0) (type default) (color 0 0 0 0))
+  )
   (wire (pts (xy 101.6 74.93) (xy 100.33 74.93))
     (stroke (width 0) (type default) (color 0 0 0 0))
   )
+  (wire (pts (xy 107.95 105.41) (xy 115.57 105.41))
+    (stroke (width 0) (type default) (color 0 0 0 0))
+  )
+  (wire (pts (xy 106.68 88.9) (xy 109.22 88.9))
+    (stroke (width 0) (type default) (color 0 0 0 0))
+  )
+  (wire (pts (xy 106.68 105.41) (xy 106.68 104.14))
+    (stroke (width 0) (type default) (color 0 0 0 0))
+  )
   (wire (pts (xy 113.03 74.93) (xy 115.57 74.93))
     (stroke (width 0) (type default) (color 0 0 0 0))
@@
     (stroke (width 0) (type default) (color 0 0 0 0))
   )
+  (wire (pts (xy 107.95 102.87) (xy 107.95 105.41))
+    (stroke (width 0) (type default) (color 0 0 0 0))
+  )
+  (wire (pts (xy 100.33 82.55) (xy 106.68 82.55))
+    (stroke (width 0) (type default) (color 0 0 0 0))
+  )
   (wire (pts (xy 77.47 113.03) (xy 77.47 116.84))
     (stroke (width 0) (type default) (color 0 0 0 0))
   )
+  (wire (pts (xy 106.68 104.14) (xy 109.22 104.14))
+    (stroke (width 0) (type default) (color 0 0 0 0))
+  )
+  (wire (pts (xy 109.22 102.87) (xy 115.57 102.87))
+    (stroke (width 0) (type default) (color 0 0 0 0))
+  )
+  (wire (pts (xy 106.68 82.55) (xy 106.68 81.28))
+    (stroke (width 0) (type default) (color 0 0 0 0))
+  )
+  (wire (pts (xy 100.33 92.71) (xy 107.95 92.71))
+    (stroke (width 0) (type default) (color 0 0 0 0))
+  )
   (wire (pts (xy 109.22 74.93) (xy 113.03 74.93))
     (stroke (width 0) (type default) (color 0 0 0 0))
   )
-  (wire (pts (xy 100.33 87.63) (xy 115.57 87.63))
+  (wire (pts (xy 107.95 92.71) (xy 107.95 95.25))
     (stroke (width 0) (type default) (color 0 0 0 0))
   )
@@
     (stroke (width 0) (type default) (color 0 0 0 0))
   )
-  (wire (pts (xy 100.33 105.41) (xy 115.57 105.41))
+  (wire (pts (xy 100.33 80.01) (xy 107.95 80.01))
     (stroke (width 0) (type default) (color 0 0 0 0))
   )
@@
     (effects (font (size 1.27 1.27)) (justify left bottom))
   )
+  (symbol (lib_id "power:PWR_FLAG") (at 46.99 73.66 0) (unit 1)
+    (in_bom yes) (on_board yes) (fields_autoplaced)
+    (property "Reference" "#FLG0102" (id 0) (at 46.99 71.755 0)
+      (effects (font (size 1.27 1.27)) hide)
+    )
+    (property "Value" "PWR_FLAG" (id 1) (at 46.99 68.58 0))
+    (property "Footprint" "" (id 2) (at 46.99 73.66 0)
+      (effects (font (size 1.27 1.27)) hide)
+    )
+    (property "Datasheet" "~" (id 3) (at 46.99 73.66 0)
+      (effects (font (size 1.27 1.27)) hide)
+    )
+    (pin "1")
+  )
   (symbol (lib_id "Mechanical:MountingHole") (at 205.74 59.69 0) (unit 1)
     (in_bom yes) (on_board yes) (fields_autoplaced)
@@
       (effects (font (size 1.27 1.27)) hide)
     )
+  )
+  (symbol (lib_id "power:PWR_FLAG") (at 34.29 73.66 0) (unit 1)
+    (in_bom yes) (on_board yes) (fields_autoplaced)
+    (property "Reference" "#FLG0101" (id 0) (at 34.29 71.755 0)
+      (effects (font (size 1.27 1.27)) hide)
+    )
+    (property "Value" "PWR_FLAG" (id 1) (at 34.29 68.58 0))
+    (property "Footprint" "" (id 2) (at 34.29 73.66 0)
+      (effects (font (size 1.27 1.27)) hide)
+    )
+    (property "Datasheet" "~" (id 3) (at 34.29 73.66 0)
+      (effects (font (size 1.27 1.27)) hide)
+    )
+    (pin "1")
+  )
+  (symbol (lib_name "+5V_1") (lib_id "power:+5V") (at 34.29 73.66 180) (unit 1)
+    (in_bom yes) (on_board yes) (fields_autoplaced)
+    (property "Reference" "#PWR0101" (id 0) (at 34.29 69.85 0)
+      (effects (font (size 1.27 1.27)) hide)
+    )
+    (property "Value" "+5V" (id 1) (at 34.29 78.74 0))
+    (property "Footprint" "" (id 2) (at 34.29 73.66 0)
+      (effects (font (size 1.27 1.27)) hide)
+    )
+    (property "Datasheet" "" (id 3) (at 34.29 73.66 0)
+      (effects (font (size 1.27 1.27)) hide)
+    )
+    (pin "1")
   )
   (symbol (lib_id "power:+5V") (at 101.6 72.39 0) (unit 1)
@@
     (pin "2")
   )
+  (symbol (lib_name "GND_1") (lib_id "power:GND") (at 46.99 73.66 0) (unit 1)
+    (in_bom yes) (on_board yes) (fields_autoplaced)
+    (property "Reference" "#PWR0102" (id 0) (at 46.99 80.01 0)
+      (effects (font (size 1.27 1.27)) hide)
+    )
+    (property "Value" "GND" (id 1) (at 46.99 78.74 0))
+    (property "Footprint" "" (id 2) (at 46.99 73.66 0)
+      (effects (font (size 1.27 1.27)) hide)
+    )
+    (property "Datasheet" "" (id 3) (at 46.99 73.66 0)
+      (effects (font (size 1.27 1.27)) hide)
+    )
+    (pin "1")
+  )
   (symbol (lib_id "Connector:USB_C_Receptacle_USB2.0") (at 85.09 90.17 0) (unit 1)
     (in_bom yes) (on_board yes) (fields_autoplaced)
@@
   )
   (symbol_instances
+    (path "/3e8b7d5c-adfc-422d-88e8-9fb76c7fd7fd"
+      (reference "#FLG0101") (unit 1) (value "PWR_FLAG") (footprint "")
+    )
+    (path "/1c0db0a9-2018-400b-a63e-06c7173005a2"
+      (reference "#FLG0102") (unit 1) (value "PWR_FLAG") (footprint "")
+    )
     (path "/482d7c41-1bff-41a0-ac76-bb30f264dec8"
       (reference "#PWR01") (unit 1) (value "+5V") (footprint "")
@@
       (reference "#PWR04") (unit 1) (value "GND") (footprint "")
     )
+    (path "/451cdb51-ec59-4bbf-9887-b12b4be048e8"
+      (reference "#PWR0101") (unit 1) (value "+5V") (footprint "")
+    )
+    (path "/e763e87b-620b-43af-b5ea-325cc0d64d6c"
+      (reference "#PWR0102") (unit 1) (value "GND") (footprint "")
+    )
     (path "/4a7e4e3b-ae39-4b0e-a125-18714ef30486"

Commit message: modif
Connections:
- net +5V: no longer names the net of J1.2 (Pin_2), J3.A4 (VBUS), J3.A9 (VBUS), J3.B4 (VBUS), J3.B9 (VBUS)
- net +5V: no longer J1.1 (Pin_1), J2.A4 (VBUS), J2.A9 (VBUS), J2.B4 (VBUS), J2.B9 (VBUS)
- new net: J1.1 (Pin_1), J2.A4 (VBUS), J2.A9 (VBUS), J2.B4 (VBUS), J2.B9 (VBUS)
Other:
- moved on the sheet: J1
Changed lines of the file:
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@@
 (kicad_sch (version 20211123) (generator eeschema)
   (paper "A4")
-  (junction (at 101.6 74.93) (diameter 0) (color 0 0 0 0)
-  )
   (junction (at 134.62 118.11) (diameter 0) (color 0 0 0 0)
   )
-  (junction (at 113.03 74.93) (diameter 0) (color 0 0 0 0)
-  )
   (junction (at 81.28 116.84) (diameter 0) (color 0 0 0 0)
   )
@@
     (stroke (width 0) (type default) (color 0 0 0 0))
   )
-  (wire (pts (xy 101.6 72.39) (xy 101.6 74.93))
-    (stroke (width 0) (type default) (color 0 0 0 0))
-  )
   (wire (pts (xy 100.33 90.17) (xy 106.68 90.17))
     (stroke (width 0) (type default) (color 0 0 0 0))
@@
     (stroke (width 0) (type default) (color 0 0 0 0))
   )
-  (wire (pts (xy 113.03 72.39) (xy 113.03 74.93))
-    (stroke (width 0) (type default) (color 0 0 0 0))
-  )
   (wire (pts (xy 109.22 92.71) (xy 115.57 92.71))
     (stroke (width 0) (type default) (color 0 0 0 0))
@@
     (stroke (width 0) (type default) (color 0 0 0 0))
   )
-  (wire (pts (xy 101.6 74.93) (xy 100.33 74.93))
+  (wire (pts (xy 100.33 74.93) (xy 106.68 74.93))
     (stroke (width 0) (type default) (color 0 0 0 0))
   )
@@
     (stroke (width 0) (type default) (color 0 0 0 0))
   )
-  (wire (pts (xy 113.03 74.93) (xy 115.57 74.93))
+  (wire (pts (xy 109.22 74.93) (xy 115.57 74.93))
     (stroke (width 0) (type default) (color 0 0 0 0))
   )
@@
     (stroke (width 0) (type default) (color 0 0 0 0))
   )
-  (wire (pts (xy 109.22 74.93) (xy 113.03 74.93))
-    (stroke (width 0) (type default) (color 0 0 0 0))
-  )
   (wire (pts (xy 107.95 92.71) (xy 107.95 95.25))
     (stroke (width 0) (type default) (color 0 0 0 0))
   )
   (wire (pts (xy 138.43 113.03) (xy 138.43 118.11))
-    (stroke (width 0) (type default) (color 0 0 0 0))
-  )
-  (wire (pts (xy 101.6 74.93) (xy 106.68 74.93))
     (stroke (width 0) (type default) (color 0 0 0 0))
   )
@@
     )
   )
-  (symbol (lib_id "power:PWR_FLAG") (at 34.29 73.66 0) (unit 1)
-    (in_bom yes) (on_board yes) (fields_autoplaced)
-    (property "Reference" "#FLG0101" (id 0) (at 34.29 71.755 0)
-      (effects (font (size 1.27 1.27)) hide)
-    )
-    (property "Value" "PWR_FLAG" (id 1) (at 34.29 68.58 0))
-    (property "Footprint" "" (id 2) (at 34.29 73.66 0)
-      (effects (font (size 1.27 1.27)) hide)
-    )
-    (property "Datasheet" "~" (id 3) (at 34.29 73.66 0)
-      (effects (font (size 1.27 1.27)) hide)
-    )
-    (pin "1")
-  )
-  (symbol (lib_name "+5V_1") (lib_id "power:+5V") (at 34.29 73.66 180) (unit 1)
-    (in_bom yes) (on_board yes) (fields_autoplaced)
-    (property "Reference" "#PWR0101" (id 0) (at 34.29 69.85 0)
-      (effects (font (size 1.27 1.27)) hide)
-    )
-    (property "Value" "+5V" (id 1) (at 34.29 78.74 0))
-    (property "Footprint" "" (id 2) (at 34.29 73.66 0)
-      (effects (font (size 1.27 1.27)) hide)
-    )
-    (property "Datasheet" "" (id 3) (at 34.29 73.66 0)
-      (effects (font (size 1.27 1.27)) hide)
-    )
-    (pin "1")
-  )
-  (symbol (lib_id "power:+5V") (at 101.6 72.39 0) (unit 1)
-    (in_bom yes) (on_board yes) (fields_autoplaced)
-    (property "Reference" "#PWR01" (id 0) (at 101.6 76.2 0)
-      (effects (font (size 1.27 1.27)) hide)
-    )
-    (property "Value" "+5V" (id 1) (at 101.6 67.31 0))
-    (property "Footprint" "" (id 2) (at 101.6 72.39 0)
-      (effects (font (size 1.27 1.27)) hide)
-    )
-    (property "Datasheet" "" (id 3) (at 101.6 72.39 0)
-      (effects (font (size 1.27 1.27)) hide)
-    )
-    (pin "1")
-  )
   (symbol (lib_id "Mechanical:MountingHole") (at 207.6247 39.1376 0) (unit 1)
     (in_bom yes) (on_board yes) (fields_autoplaced)
@@
       (effects (font (size 1.27 1.27)) hide)
     )
-  )
-  (symbol (lib_id "power:+5V") (at 113.03 72.39 0) (unit 1)
-    (in_bom yes) (on_board yes) (fields_autoplaced)
-    (property "Reference" "#PWR02" (id 0) (at 113.03 76.2 0)
-      (effects (font (size 1.27 1.27)) hide)
-    )
-    (property "Value" "+5V" (id 1) (at 113.03 67.31 0))
-    (property "Footprint" "" (id 2) (at 113.03 72.39 0)
-      (effects (font (size 1.27 1.27)) hide)
-    )
-    (property "Datasheet" "" (id 3) (at 113.03 72.39 0)
-      (effects (font (size 1.27 1.27)) hide)
-    )
-    (pin "1")
   )
   (symbol (lib_id "Mechanical:MountingHole") (at 212.1933 51.155 0) (unit 1)
@@
     (pin "1")
   )
-  (symbol (lib_id "Connector_Generic:Conn_01x02") (at 109.22 41.91 270) (mirror x) (unit 1)
+  (symbol (lib_id "Connector_Generic:Conn_01x02") (at 106.68 41.91 90) (unit 1)
     (in_bom yes) (on_board yes) (fields_autoplaced)
     (property "Reference" "J1" (id 0) (at 111.76 40.6399 90)
-      (effects (font (size 1.27 1.27)) (justify left))
+      (effects (font (size 1.27 1.27)) (justify right))
     )
     (property "Value" "Conn_01x02" (id 1) (at 111.76 43.1799 90)
-      (effects (font (size 1.27 1.27)) (justify left))
-    )
-    (property "Footprint" "Connector_JST:JST_XH_B2B-XH-A_1x02_P2.50mm_Vertical" (id 2) (at 109.22 41.91 0)
-      (effects (font (size 1.27 1.27)) hide)
-    )
-    (property "Datasheet" "~" (id 3) (at 109.22 41.91 0)
+      (effects (font (size 1.27 1.27)) (justify right))
+    )
+    (property "Footprint" "Connector_JST:JST_XH_B2B-XH-A_1x02_P2.50mm_Vertical" (id 2) (at 106.68 41.91 0)
+      (effects (font (size 1.27 1.27)) hide)
+    )
+    (property "Datasheet" "~" (id 3) (at 106.68 41.91 0)
       (effects (font (size 1.27 1.27)) hide)
     )
@@
   )
   (symbol_instances
-    (path "/3e8b7d5c-adfc-422d-88e8-9fb76c7fd7fd"
-      (reference "#FLG0101") (unit 1) (value "PWR_FLAG") (footprint "")
-    )
     (path "/1c0db0a9-2018-400b-a63e-06c7173005a2"
       (reference "#FLG0102") (unit 1) (value "PWR_FLAG") (footprint "")
     )
-    (path "/482d7c41-1bff-41a0-ac76-bb30f264dec8"
-      (reference "#PWR01") (unit 1) (value "+5V") (footprint "")
-    )
-    (path "/82319c6a-c8f2-4bc4-8446-e48c4948afc3"
-      (reference "#PWR02") (unit 1) (value "+5V") (footprint "")
-    )
     (path "/c319fcc3-e5bf-4d03-ab1c-f15ea771e946"
       (reference "#PWR03") (unit 1) (value "GND") (footprint "")
@@
       (reference "#PWR04") (unit 1) (value "GND") (footprint "")
     )
-    (path "/451cdb51-ec59-4bbf-9887-b12b4be048e8"
-      (reference "#PWR0101") (unit 1) (value "+5V") (footprint "")
-    )
     (path "/e763e87b-620b-43af-b5ea-325cc0d64d6c"
